File: hardware/lite-foc/lite-foc.kicad_sch (KiCad schematic)
At the start: 30 parts, among them J1 USB_C_Receptacle_USB2.0_16P, U1 STM32F411CEUx, U2 DRV8313PWP, U3 INA240A2PW, U4 INA240A2PW, Y1 8M

Commit message: feat:原理图绘制完成 初步开始layout
Parts:
- removed S1: SW-PB, mylib:SMD_6X6X4.3, symbol my_lib:SW-PB
- removed U2: DRV8313PWP, Package_SO:HTSSOP-28-1EP_4.4x9.7mm_P0.65mm_EP2.75x6.2mm, symbol my_lib:DRV8313PWP
- added C13: 100K, Capacitor_SMD:C_0805_2012Metric, symbol Device:C
- added C14, C15, C19, C21: 0.1uF, Capacitor_SMD:C_0805_2012Metric, symbol Device:C
- added C16, C17, C20, C22: 100uF, Capacitor_SMD:C_0805_2012Metric, symbol Device:C
- added C18, C23, C24, C25: 10uF, Capacitor_SMD:C_0805_2012Metric, symbol Device:C
- added C26: 100uf, Capacitor_SMD:C_0805_2012Metric, symbol Device:C
- added D1: SS54, Diode_SMD:D_SMA, symbol PCM_Diode_Schottky_AKL:SS54
- added D2: LED, LED_SMD:LED_0805_2012Metric, symbol Device:LED
- added D3: SMBJ5.0CA, Diode_SMD:D_SMA, symbol PCM_Diode_TVS_AKL:SMBJ5.0CA
- added D4, D5, D6: B5817WS, Diode_SMD:D_SOD-323, symbol Device:D
- added J2: Conn_01x02_MountingPin, Connector_JST:JST_SHL_SM02B-SHLS-TF_1x02-1MP_P1.00mm_Horizontal, symbol Connector_Generic_MountingPin:Conn_01x02_MountingPin
- added J3: Conn_01x03, Connector_AMASS:AMASS_MR30PW-M_1x03_P3.50mm_Horizontal, symbol Connector_Generic:Conn_01x03
- added J4: Conn_01x03_MountingPin, Connector_JST:JST_SH_BM03B-SRSS-TB_1x03-1MP_P1.00mm_Vertical, symbol Connector_Generic_MountingPin:Conn_01x03_MountingPin
- added J5: Conn_01x02, Connector_AMASS:AMASS_XT30PW-M_1x02_P2.50mm_Horizontal, symbol Connector_Generic:Conn_01x02
- added L1: 6.8uH, Inductor_SMD:L_0805_2012Metric, symbol Device:L
- added R10: 1.5K, Resistor_SMD:R_0805_2012Metric, symbol Device:R
- added R11: 10K, PCM_Resistor_SMD_AKL:R_0805_2012Metric, symbol Device:R
- added R12: 2K, PCM_Resistor_SMD_AKL:R_0805_2012Metric, symbol Device:R
- added R13: 1M, PCM_Resistor_SMD_AKL:R_0805_2012Metric, symbol Device:R
- added R3: 120, Resistor_SMD:R_0805_2012Metric, symbol Device:R
- added R7, R8: 22, Resistor_SMD:R_0805_2012Metric, symbol Device:R
- added R9: 1.8K, PCM_Resistor_SMD_AKL:R_0805_2012Metric, symbol Device:R
- added SW1: CK_KMS2xxG, Button_Switch_SMD:SW_SPST_CK_KMS2xxG, symbol Switch:CK_KMS2xxG
- added U3: SN65HVD232, Package_SO:SOIC-8_3.9x4.9mm_P1.27mm, symbol Interface_CAN_LIN:SN65HVD232
- added U5: LP2992 3V3, PCM_Package_TO_SOT_SMD_AKL:SOT-23-5, symbol my_lib:LP2992_3V3
- added U6: ME3116, PCM_Package_TO_SOT_SMD_AKL:SOT-23-6, symbol my_lib:ME3116
- added U7: DRV8313PWP, Package_SO:HTSSOP-28-1EP_4.4x9.7mm_P0.65mm_EP3.4x9.5mm_Mask2.4x6.17mm, symbol my_lib:DRV8313PWP
- C1: renamed from C2; footprint (none) -> Capacitor_SMD:C_0805_2012Metric
- C10: renamed from C8; footprint (none) -> Capacitor_SMD:C_0805_2012Metric
- C11: renamed from C9; footprint (none) -> Capacitor_SMD:C_0805_2012Metric
- C12: renamed from C3; footprint (none) -> Capacitor_SMD:C_0805_2012Metric
- C2: renamed from C1; footprint (none) -> Capacitor_SMD:C_0805_2012Metric
- C27: renamed from C13; footprint (none) -> Capacitor_SMD:C_0805_2012Metric
- C28: renamed from C14; footprint (none) -> Capacitor_SMD:C_0805_2012Metric
- C29: renamed from C15; footprint (none) -> Capacitor_SMD:C_0805_2012Metric
- C3: renamed from C4; footprint (none) -> Capacitor_SMD:C_0805_2012Metric
- C4: renamed from C10; value C -> 0.1uF; footprint (none) -> Capacitor_SMD:C_0805_2012Metric
- C5: renamed from C11; value C -> 0.1uF; footprint (none) -> Capacitor_SMD:C_0805_2012Metric
- C6: renamed from C5; footprint (none) -> Capacitor_SMD:C_0805_2012Metric
- C7: renamed from C6; footprint (none) -> Capacitor_SMD:C_0805_2012Metric
- C8: renamed from C12; footprint (none) -> Capacitor_SMD:C_0805_2012Metric
- C9: renamed from C7; footprint (none) -> Capacitor_SMD:C_0805_2012Metric
- J1: footprint Connector_USB:USB_C_Receptacle_G-Switch_GT-USB-7010ASV -> Connector_USB:USB_C_Receptacle_GCT_USB4105-xx-A_16P_TopMnt_Horizontal
- R1: renamed from R2; value 0.0.1 -> 0.01; footprint (none) -> Resistor_SMD:R_0805_2012Metric
- R14: renamed from R8; footprint (none) -> Resistor_SMD:R_0805_2012Metric
- R15: renamed from R5; footprint (none) -> Resistor_SMD:R_0805_2012Metric
- R16: renamed from R7; footprint (none) -> Resistor_SMD:R_0805_2012Metric
- R2: renamed from R3; footprint (none) -> Resistor_SMD:R_0805_2012Metric
- R4: renamed from R6; footprint (none) -> Resistor_SMD:R_0805_2012Metric
- R5: renamed from R4; footprint (none) -> Resistor_SMD:R_0805_2012Metric
- R6: renamed from R1; footprint (none) -> Resistor_SMD:R_0805_2012Metric
- U4: renamed from U1; footprint Package_DFN_QFN:QFN-48-1EP_7x7mm_P0.5mm_EP5.6x5.6mm -> Package_DFN_QFN:QFN-48-1EP_7x7mm_P0.5mm_EP5.15x5.15mm
- renumbered U3 to U1, U4 to U2
Connections:
- net +3.3VA is gone; now on net +3.3V: C10.1, C11.1, R4.1, U4.9 (VDDA)
- net +3.3V: now also C19.1, C23.1, U3.3 (VCC), U5.5 (VOUT)
- net DRV_EN: now also U4.25 (PB12), U7.22 (EN3), U7.24 (EN2), U7.26 (EN1)
- net DRV_FAULT: now also U7.18 (NFAULT)
- net GND: now also C16.2, C17.2, C18.2, C19.2, C20.2, C21.1, C22.2, C23.2, C24.1, C25.1, C26.2, D3.1 (K), D5.2 (A), J2.MP (MountPin), J4.2 (Pin_2), J4.MP (MountPin), J5.2 (Pin_2), R12.2, R9.2, SW1.2, SW1.SH (B), U3.2 (GND), U5.2 (GND), U6.2 (GND), U7.10 (PGND3), U7.12 (COMPP), U7.13 (COMPN), U7.14 (GND), U7.20 (GND), U7.28 (GND), U7.29 (TH_PAD), U7.6 (PGND1), U7.7 (PGND2)
- net MOTOR_A: now also J3.1 (Pin_1)
- net MOTOR_A_CS: now also U7.5 (OUT1)
- net MOTOR_B: now also J3.2 (Pin_2)
- net MOTOR_B_CS: now also U7.8 (OUT2)
- net MOTOR_C: now also J3.3 (Pin_3), U7.9 (OUT3)
- net NRST: now also SW1.1
- net PWM_A: now also U4.40 (PB4), U7.27 (IN1)
- net PWM_B: now also U4.41 (PB5), U7.25 (IN2)
- net PWM_C: now also U4.18 (PB0), U7.23 (IN3)
- net SENSE_A: now also U4.10 (PA0)
- net SENSE_B: now also U4.11 (PA1)
- net USB_DM_IN: now also R7.1
- net USB_DP: now also R10.1, R8.2
- net USB_DP_IN: now also R8.1
- net V3P3: now also U7.16 (NRESET), U7.17 (NSLEEP)
- net VBUS: now also D4.2 (A), R10.2
- net VCC: now also C16.1, C17.1, C20.1, C22.1, C26.1, D1.1 (K), D3.2 (A), D6.2 (A), U7.11 (VM2), U7.4 (VM1)
- net at C27.1: now also U7.1 (CPL)
- net at C27.2: now also U7.2 (CPH)
- net at C29.1: now also U7.15 (V3P3)
- net at C28.1: now also U7.3 (VCP)
- net Encoder_PWM: now reaches U4.30 (PA9)
- net Encoder_PWM: now also J4.1 (Pin_1)
- net CAN_D: now reaches U4.45 (PB8)
- net CAN_D: now also U3.1 (D)
- net CAN_R: now reaches U4.46 (PB9)
- net CAN_R: now also U3.4 (R)
- net USB_DN renamed USB_DM
- net USB_DM: now also R7.2
- new net: D5.1 (K), U6.6 (SW)
- new net: D2.1 (K), R12.1
- new net: C14.1, C15.1, U6.1 (BS)
- new net: C14.2, C15.2, L1.1
- new net: C24.2, D6.1 (K), R13.2, U6.5 (IN)
- new net: C18.1, U5.4 (BYPASS)
- new net: C13.2, R11.2, R9.1, U6.3 (FB)
- new net: R13.1, U6.4 (EN)
- new net +5V: C13.1, C21.2, C25.2, D2.2 (A), D4.1 (K), J4.3 (Pin_3), L1.2, R11.1, U5.1 (VIN), U5.3 (ON/OFF)
- new net CAN_H: J2.1 (Pin_1), R3.1, U3.7 (CANH)
- new net CAN_L: J2.2 (Pin_2), R3.2, U3.6 (CANL)
- new net VCC_IN: D1.2 (A), J5.1 (Pin_1)
- no-connect marks 0 -> 26
Other:
- note added: "CAN"
- note added: "COM"
- note added: "POWER"
- note added: "PWM"
- moved on the sheet: C1, C10, C11, C12, C2, C27, C28, C29, C3, C4, C5, C6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
